Commit message: attached the charge model file to the end effector of the robot. I directly commit, plz resolve the conflict if there are some..

File: ur_description/urdf/ur5.urdf.xacro (robot description, xacro)
@@ -284,4 +284,14 @@
     </joint>
     <link name="${prefix}ee_link">
+  <!-- chen add -->
+         <visual>
+        <geometry>
+          <mesh filename="package://ur_description/meshes/ee/chargeattachment.dae" />
+        </geometry>
+        <material name="blue">
+          <color rgba="0.0 0.0 0.8 1.0"/>
+        </material>
+      </visual>
+   <!-- add the mesh to the end effector -->
       <collision>
         <geometry>

File: ur_description/urdf/ur5_robot.urdf.xacro (robot description, xacro)
@@ -17,5 +17,5 @@
     </geometry>
      <material name="LightGrey">
-       <color rgba="0.7 0.7 0.7 1.0"/>
+       <color rgba="0.5 0.5 0.5 1.0"/>
      </material>
    </visual>

Commit message: Use better names for links and joints
world_{link,joint,controller} -> lateral_slider_*
x_{link,joint,controller} -> forward_slider_*

Some doc says <virtual_joint> is not required if the root link
is fixed. It's still a question if that is true.

File: ur_description/urdf/ur5.urdf.xacro (robot description, xacro)
@@ -281,9 +281,11 @@
       <parent link="${prefix}wrist_3_link" />
       <child link = "${prefix}ee_link" />
-      <origin xyz="0.0 ${wrist_3_length} 0.0" rpy="0.0 0.0 ${pi/2.0}" />
+      <origin xyz="0.0 ${wrist_3_length} 0.0" rpy="${-pi/2.0} 0.0 0.0" />
     </joint>
     <link name="${prefix}ee_link">
   <!-- chen add -->
-         <visual>
+      <visual>
+        <!-- Uses -pi/2 pitch such that z axis points outwards. -->
+        <origin xyz="0 0 0" rpy="0 ${-pi/2.0} 0"/>
         <geometry>
           <mesh filename="package://ur_description/meshes/ee/chargeattachment.dae" />
@@ -296,7 +298,7 @@
       <collision>
         <geometry>
-          <box size="0.01 0.01 0.01"/>
-        </geometry>
-        <origin rpy="0 0 0" xyz="-0.01 0 0"/>
+          <cylinder radius="0.04" length="0.005"/>
+        </geometry>
+        <origin rpy="0 0 0" xyz="0 0 0.0025"/>
       </collision>
     </link>

File: ur_description/urdf/ur5_joint_limited_robot.urdf.xacro (robot description, xacro)
@@ -15,19 +15,15 @@
     wrist_3_lower_limit="${-pi}" wrist_3_upper_limit="${pi}"
   />
-  <link name="world" >
+  <link name="world">
     <static>true</static>
-    <origin xyz="0.0 0.0 0.0" rpy="0.0 0.0 0.0" />
-    </link>
- <link name="y_link" >
-      <inertial>
-      <mass value="0.01" />
-      <origin xyz="0 0 0" rpy="0 -0 0"/>
-      <inertia ixx="0.01" ixy="0" ixz="0" iyy="0.01" iyz="0" izz="0.01"/>
-    </inertial>
   </link>
-  <link name="x_link">
+  <joint name="world_joint" type="fixed">
+    <parent link="world" />
+    <child link="lateral_slider_link" />
+  </joint>
+  <link name="lateral_slider_link" >
    <visual>
     <geometry>
-        <box size="3.0 0.04 0.01"/>
+        <box size="0.05 12 0.01"/>
     </geometry>
      <material name="LightGrey">
@@ -41,26 +37,36 @@
     </inertial>
   </link>
-  <joint name="worldfix_joint" type="fixed">
-    <parent link="world" />
-    <child link = "y_link" />
-    <origin xyz="0.0 0.0 0.0" rpy="0.0 0.0 0.0" />
-  </joint>
-  <joint name="world_joint" type="prismatic">
-    <parent link="y_link" />
-    <child link = "x_link" />
+  <link name="forward_slider_link">
+   <visual>
+    <geometry>
+        <box size="3.0 0.05 0.01"/>
+    </geometry>
+     <material name="LightGrey">
+       <color rgba="0.7 0.7 0.7 1.0"/>
+     </material>
+   </visual>
+    <inertial>
+      <mass value="0.01" />
+      <origin xyz="0 0 0" rpy="0 -0 0"/>
+      <inertia ixx="0.01" ixy="0" ixz="0" iyy="0.01" iyz="0" izz="0.01"/>
+    </inertial>
+  </link>
+  <joint name="lateral_slider_joint" type="prismatic">
+    <parent link="lateral_slider_link" />
+    <child link="forward_slider_link" />
     <origin xyz="0.0 0.0 0.0" rpy="0.0 0.0 0.0" />
     <axis xyz="0 1 0" />
-    <limit effort="3000" velocity="20.0" lower="-10" upper="10" />
+    <limit effort="3000" velocity="20.0" lower="-6" upper="6" />
   </joint>
-  <joint name="x_joint" type="prismatic">
-    <parent link="x_link" />
-    <child link = "base_link" />
+  <joint name="forward_slider_joint" type="prismatic">
+    <parent link="forward_slider_link" />
+    <child link="base_link" />
     <origin xyz="0.0 0.0 0.0" rpy="0.0 0.0 0.0" />
     <axis xyz="1 0 0" />
-    <limit effort="3000" velocity="20.0" lower="-3" upper="3" />
+    <limit effort="3000" velocity="20.0" lower="-1.5" upper="1.5" />
   </joint>
-  <transmission name="world_joint_trans">
+  <transmission name="lateral_slider_joint_trans">
     <type>transmission_interface/SimpleTransmission</type>
-    <joint name="world_joint">
+    <joint name="lateral_slider_joint">
       <hardwareInterface>hardware_interface/EffortJointInterface</hardwareInterface>
     </joint>
@@ -69,7 +75,7 @@
     </actuator>
   </transmission>
-  <transmission name="x_joint_trans">
+  <transmission name="forward_slider_joint_trans">
     <type>transmission_interface/SimpleTransmission</type>
-    <joint name="x_joint">
+    <joint name="forward_slider_joint">
       <hardwareInterface>hardware_interface/EffortJointInterface</hardwareInterface>
     </joint>
