Commit message: add two joints and controllers to realize the sliding on certain axis. The world_controller allows the arm base to move in Y axis, The x_controller allows the arm base to move in X axis, by directly publish the controller command.
TODOLIST:
 add the charge mount to the end effector of the UR5..
 try to control the ur5 automatically.

File: ur_description/urdf/ur5_joint_limited_robot.urdf.xacro (robot description, xacro)
@@ -15,9 +15,53 @@
     wrist_3_lower_limit="${-pi}" wrist_3_upper_limit="${pi}"
   />
-  <link name="world" />
-  <joint name="world_joint" type="fixed">
+  <link name="world" >
+    <origin xyz="0.0 0.0 0.0" rpy="0.0 0.0 0.0" />
+    </link>
+  <link name="x_link">
+   <visual>
+    <geometry>
+        <box size="2.0 0.2 0.02"/>
+    </geometry>
+     <material name="LightGrey">
+       <color rgba="0.7 0.7 0.7 1.0"/>
+     </material>
+   </visual>
+    <inertial>
+      <mass value="0.01" />
+      <origin xyz="0 0 0" rpy="0 -0 0"/>
+      <inertia ixx="0.01" ixy="0" ixz="0" iyy="0.01" iyz="0" izz="0.01"/>
+    </inertial>
+  </link>
+  <joint name="world_joint" type="prismatic">
     <parent link="world" />
+    <child link = "x_link" />
+    <origin xyz="0.0 0.0 0.0" rpy="0.0 0.0 0.0" />
+    <axis xyz="0 1 0" />
+    <limit effort="3000" velocity="20.0" lower="-100" upper="100" />
+  </joint>
+  <joint name="x_joint" type="prismatic">
+    <parent link="x_link" />
     <child link = "base_link" />
     <origin xyz="0.0 0.0 0.0" rpy="0.0 0.0 0.0" />
+    <axis xyz="1 0 0" />
+    <limit effort="3000" velocity="20.0" lower="-100" upper="100" />
   </joint>
+  <transmission name="world_joint_trans">
+    <type>transmission_interface/SimpleTransmission</type>
+    <joint name="world_joint">
+      <hardwareInterface>hardware_interface/EffortJointInterface</hardwareInterface>
+    </joint>
+    <actuator name="$foo_motor">
+      <mechanicalReduction>1</mechanicalReduction>
+    </actuator>
+  </transmission>
+  <transmission name="x_joint_trans">
+    <type>transmission_interface/SimpleTransmission</type>
+    <joint name="x_joint">
+      <hardwareInterface>hardware_interface/EffortJointInterface</hardwareInterface>
+    </joint>
+    <actuator name="$foo1_motor">
+      <mechanicalReduction>1</mechanicalReduction>
+    </actuator>
+  </transmission>
 </robot>

File: ur_description/urdf/ur5_robot.urdf.xacro (robot description, xacro)
@@ -8,9 +8,53 @@
   <!-- arm -->
   <xacro:ur5_robot prefix="" joint_limited="false"/>
-  <link name="world" />
-  <joint name="world_joint" type="fixed">
+  <link name="world" >
+    <origin xyz="0.0 0.0 0.0" rpy="0.0 0.0 0.0" />
+    </link>
+  <link name="x_link">
+   <visual>
+    <geometry>
+        <box size="2.0 0.2 0.02"/>
+    </geometry>
+     <material name="LightGrey">
+       <color rgba="0.7 0.7 0.7 1.0"/>
+     </material>
+   </visual>
+    <inertial>
+      <mass value="0.01" />
+      <origin xyz="0 0 0" rpy="0 -0 0"/>
+      <inertia ixx="0.01" ixy="0" ixz="0" iyy="0.01" iyz="0" izz="0.01"/>
+    </inertial>
+  </link>
+  <joint name="world_joint" type="prismatic">
     <parent link="world" />
+    <child link = "x_link" />
+    <origin xyz="0.0 0.0 0.0" rpy="0.0 0.0 0.0" />
+    <axis xyz="0 1 0" />
+    <limit effort="3000" velocity="10.0" lower="-100" upper="100" />
+  </joint>
+  <joint name="x_joint" type="prismatic">
+    <parent link="x_link" />
     <child link = "base_link" />
     <origin xyz="0.0 0.0 0.0" rpy="0.0 0.0 0.0" />
+    <axis xyz="1 0 0" />
+    <limit effort="3000" velocity="10.0" lower="-100" upper="100" />
   </joint>
+  <transmission name="world_joint_trans">
+    <type>transmission_interface/SimpleTransmission</type>
+    <joint name="world_joint">
+      <hardwareInterface>hardware_interface/EffortJointInterface</hardwareInterface>
+    </joint>
+    <actuator name="$foo_motor">
+      <mechanicalReduction>1</mechanicalReduction>
+    </actuator>
+  </transmission>
+  <transmission name="x_joint_trans">
+    <type>transmission_interface/SimpleTransmission</type>
+    <joint name="x_joint">
+      <hardwareInterface>hardware_interface/EffortJointInterface</hardwareInterface>
+    </joint>
+    <actuator name="$foo1_motor">
+      <mechanicalReduction>1</mechanicalReduction>
+    </actuator>
+  </transmission>
 </robot>

Commit message: Connect x_link world_link controllers to UR5

File: ur_description/urdf/ur5_joint_limited_robot.urdf.xacro (robot description, xacro)
@@ -21,5 +21,5 @@
    <visual>
     <geometry>
-        <box size="2.0 0.2 0.02"/>
+        <box size="3.0 0.04 0.01"/>
     </geometry>
      <material name="LightGrey">
@@ -38,5 +38,5 @@
     <origin xyz="0.0 0.0 0.0" rpy="0.0 0.0 0.0" />
     <axis xyz="0 1 0" />
-    <limit effort="3000" velocity="20.0" lower="-100" upper="100" />
+    <limit effort="3000" velocity="20.0" lower="-10" upper="10" />
   </joint>
   <joint name="x_joint" type="prismatic">
@@ -45,5 +45,5 @@
     <origin xyz="0.0 0.0 0.0" rpy="0.0 0.0 0.0" />
     <axis xyz="1 0 0" />
-    <limit effort="3000" velocity="20.0" lower="-100" upper="100" />
+    <limit effort="3000" velocity="20.0" lower="-3" upper="3" />
   </joint>
   <transmission name="world_joint_trans">

Commit message: solve the world frame moving problem.. reason:  world link not fixed.

File: ur_description/urdf/ur5_joint_limited_robot.urdf.xacro (robot description, xacro)
@@ -16,6 +16,14 @@
   />
   <link name="world" >
+    <static>true</static>
     <origin xyz="0.0 0.0 0.0" rpy="0.0 0.0 0.0" />
     </link>
+ <link name="y_link" >
+      <inertial>
+      <mass value="0.01" />
+      <origin xyz="0 0 0" rpy="0 -0 0"/>
+      <inertia ixx="0.01" ixy="0" ixz="0" iyy="0.01" iyz="0" izz="0.01"/>
+    </inertial>
+  </link>
   <link name="x_link">
    <visual>
@@ -33,6 +41,11 @@
     </inertial>
   </link>
+  <joint name="worldfix_joint" type="fixed">
+    <parent link="world" />
+    <child link = "y_link" />
+    <origin xyz="0.0 0.0 0.0" rpy="0.0 0.0 0.0" />
+  </joint>
   <joint name="world_joint" type="prismatic">
-    <parent link="world" />
+    <parent link="y_link" />
     <child link = "x_link" />
     <origin xyz="0.0 0.0 0.0" rpy="0.0 0.0 0.0" />

Commit message: add xy planner... change some parameters like the gain and collision. now seems no drifting..
using a new branch ...

File: ur_description/urdf/ur5_joint_limited_robot.urdf.xacro (robot description, xacro)
@@ -29,5 +29,5 @@
    <visual>
     <geometry>
-        <box size="3.0 0.04 0.01"/>
+        <box size="2.5 0.04 0.01"/>
     </geometry>
      <material name="LightGrey">
@@ -51,5 +51,5 @@
     <origin xyz="0.0 0.0 0.0" rpy="0.0 0.0 0.0" />
     <axis xyz="0 1 0" />
-    <limit effort="3000" velocity="20.0" lower="-10" upper="10" />
+    <limit effort="10000" velocity="20.0" lower="-10" upper="10" />
   </joint>
   <joint name="x_joint" type="prismatic">
@@ -58,5 +58,5 @@
     <origin xyz="0.0 0.0 0.0" rpy="0.0 0.0 0.0" />
     <axis xyz="1 0 0" />
-    <limit effort="3000" velocity="20.0" lower="-3" upper="3" />
+    <limit effort="10000" velocity="20.0" lower="-3" upper="3" />
   </joint>
   <transmission name="world_joint_trans">

File: ur_description/urdf/ur5_robot.urdf.xacro (robot description, xacro)
@@ -21,5 +21,5 @@
    <visual>
     <geometry>
-        <box size="2.0 0.2 0.02"/>
+        <box size="2.5 0.04 0.01"/>
     </geometry>
      <material name="LightGrey">
@@ -43,5 +43,5 @@
     <origin xyz="0.0 0.0 0.0" rpy="0.0 0.0 0.0" />
     <axis xyz="0 1 0" />
-    <limit effort="3000" velocity="10.0" lower="-100" upper="100" />
+    <limit effort="10000" velocity="10.0" lower="-100" upper="100" />
   </joint>
   <joint name="x_joint" type="prismatic">
@@ -50,5 +50,5 @@
     <origin xyz="0.0 0.0 0.0" rpy="0.0 0.0 0.0" />
     <axis xyz="1 0 0" />
-    <limit effort="3000" velocity="10.0" lower="-100" upper="100" />
+    <limit effort="10000" velocity="10.0" lower="-100" upper="100" />
   </joint>
   <transmission name="world_joint_trans">

Commit message: resolve the conflict. increased the real-time factor

File: ur_description/urdf/ur5_joint_limited_robot.urdf.xacro (robot description, xacro)
@@ -23,12 +23,4 @@
   </joint>
   <link name="lateral_slider_link" >
-   <visual>
-    <geometry>
-        <box size="0.05 12 0.01"/>
-    </geometry>
-     <material name="LightGrey">
-       <color rgba="0.7 0.7 0.7 1.0"/>
-     </material>
-   </visual>
     <inertial>
       <mass value="0.01" />

File: ur_description/urdf/ur5_robot.urdf.xacro (robot description, xacro)
@@ -8,9 +8,13 @@
   <!-- arm -->
   <xacro:ur5_robot prefix="" joint_limited="false"/>
-  <link name="world" >
-    <origin xyz="0.0 0.0 0.0" rpy="0.0 0.0 0.0" />
+  <link name="world">
+    <static>true</static>
   </link>
-  <link name="y_link" >
-      <inertial>
+  <joint name="world_joint" type="fixed">
+    <parent link="world" />
+    <child link="lateral_slider_link" />
+  </joint>
+  <link name="lateral_slider_link" >
+    <inertial>
       <mass value="0.01" />
       <origin xyz="0 0 0" rpy="0 -0 0"/>
@@ -18,11 +22,11 @@
     </inertial>
   </link>
-  <link name="x_link">
+  <link name="forward_slider_link">
    <visual>
     <geometry>
-        <box size="2.5 0.04 0.01"/>
+        <box size="3.0 0.05 0.01"/>
     </geometry>
      <material name="LightGrey">
-       <color rgba="0.5 0.5 0.5 1.0"/>
+       <color rgba="0.7 0.7 0.7 1.0"/>
      </material>
    </visual>
@@ -33,26 +37,21 @@
     </inertial>
   </link>
-  <joint name="worldfix_joint" type="fixed">
-    <parent link="world" />
-    <child link = "y_link" />
-    <origin xyz="0.0 0.0 0.0" rpy="0.0 0.0 0.0" />
-  </joint>
-  <joint name="world_joint" type="prismatic">
-    <parent link="y_link" />
-    <child link = "x_link" />
+  <joint name="lateral_slider_joint" type="prismatic">
+    <parent link="lateral_slider_link" />
+    <child link="forward_slider_link" />
     <origin xyz="0.0 0.0 0.0" rpy="0.0 0.0 0.0" />
     <axis xyz="0 1 0" />
-    <limit effort="10000" velocity="10.0" lower="-100" upper="100" />
+    <limit effort="10000" velocity="20.0" lower="-10" upper="10" />
   </joint>
-  <joint name="x_joint" type="prismatic">
-    <parent link="x_link" />
-    <child link = "base_link" />
+  <joint name="forward_slider_joint" type="prismatic">
+    <parent link="forward_slider_link" />
+    <child link="base_link" />
     <origin xyz="0.0 0.0 0.0" rpy="0.0 0.0 0.0" />
     <axis xyz="1 0 0" />
-    <limit effort="10000" velocity="10.0" lower="-100" upper="100" />
+    <limit effort="10000" velocity="20.0" lower="-1.5" upper="1.5" />
   </joint>
-  <transmission name="world_joint_trans">
+  <transmission name="lateral_slider_joint_trans">
     <type>transmission_interface/SimpleTransmission</type>
-    <joint name="world_joint">
+    <joint name="lateral_slider_joint">
       <hardwareInterface>hardware_interface/EffortJointInterface</hardwareInterface>
     </joint>
@@ -61,7 +60,7 @@
     </actuator>
   </transmission>
-  <transmission name="x_joint_trans">
+  <transmission name="forward_slider_joint_trans">
     <type>transmission_interface/SimpleTransmission</type>
-    <joint name="x_joint">
+    <joint name="forward_slider_joint">
       <hardwareInterface>hardware_interface/EffortJointInterface</hardwareInterface>
     </joint>

Commit message: Fix typos

File: ur_description/urdf/ur5_joint_limited_robot.urdf.xacro (robot description, xacro)
@@ -23,4 +23,12 @@
   </joint>
   <link name="lateral_slider_link" >
+   <visual>
+    <geometry>
+        <box size="0.05 20 0.01"/>
+    </geometry>
+     <material name="LightGrey">
+       <color rgba="0.7 0.7 0.7 1.0"/>
+     </material>
+   </visual>
     <inertial>
       <mass value="0.01" />

Commit message: the lateral model is too long..change to 15 meters

File: ur_description/urdf/ur5_joint_limited_robot.urdf.xacro (robot description, xacro)
@@ -25,5 +25,5 @@
    <visual>
     <geometry>
-        <box size="0.05 20 0.01"/>
+        <box size="0.05 15 0.01"/>
     </geometry>
      <material name="LightGrey">

Commit message: add realsense plugin

File: ur_description/urdf/ur5_joint_limited_robot.urdf.xacro (robot description, xacro)
@@ -66,4 +66,15 @@
     <limit effort="10000" velocity="20.0" lower="-1.5" upper="1.5" />
   </joint>
+  <!-- chen add -->
+  <xacro:include filename="$(find realsense_gazebo_plugin)/urdf/realsense-RS200.macro.xacro"/>
+  <!-- Gazebo world link required to position the robot with respect to origin -->
+  <!-- Place camera referenced to world frame -->
+  <joint name="realsense_joint" type="fixed">
+    <parent link="ee_link"/>
+    <child link="rs200_camera"/>
+    <origin rpy="${pi/-2.0} ${pi/-2.0} 0" xyz="0 0.04 -0.004"/>
+  </joint>
+  <xacro:realsense-rs200/>
+    <!-- chen add -->
   <transmission name="lateral_slider_joint_trans">
     <type>transmission_interface/SimpleTransmission</type>

Commit message: 0801

File: ur_description/urdf/ur5_joint_limited_robot.urdf.xacro (robot description, xacro)
@@ -25,5 +25,5 @@
    <visual>
     <geometry>
-        <box size="0.05 15 0.01"/>
+        <box size="0.05 15 0.02"/>
     </geometry>
      <material name="LightGrey">
@@ -40,5 +40,5 @@
    <visual>
     <geometry>
-        <box size="3.0 0.05 0.01"/>
+        <box size="5.0 0.05 0.02"/>
     </geometry>
      <material name="LightGrey">
@@ -73,5 +73,5 @@
     <parent link="ee_link"/>
     <child link="rs200_camera"/>
-    <origin rpy="${pi/-2.0} ${pi/-2.0} 0" xyz="0 0.04 -0.004"/>
+    <origin rpy="${pi/-2.0} ${pi/-2.0} 0" xyz="0 0.06 -0.004"/>
   </joint>
   <xacro:realsense-rs200/>

Commit message: 0817

File: ur_description/urdf/ur5_joint_limited_robot.urdf.xacro (robot description, xacro)
@@ -40,5 +40,5 @@
    <visual>
     <geometry>
-        <box size="5.0 0.05 0.02"/>
+        <box size="6.0 0.1 0.03"/>
     </geometry>
      <material name="LightGrey">
@@ -47,7 +47,7 @@
    </visual>
     <inertial>
-      <mass value="0.01" />
+      <mass value="100" />
       <origin xyz="0 0 0" rpy="0 -0 0"/>
-      <inertia ixx="0.01" ixy="0" ixz="0" iyy="0.01" iyz="0" izz="0.01"/>
+      <inertia ixx="0.1" ixy="0" ixz="0" iyy="0.1" iyz="0" izz="0.1"/>
     </inertial>
   </link>
@@ -64,5 +64,5 @@
     <origin xyz="0.0 0.0 0.0" rpy="0.0 0.0 0.0" />
     <axis xyz="1 0 0" />
-    <limit effort="10000" velocity="20.0" lower="-1.5" upper="1.5" />
+    <limit effort="3000" velocity="10.0" lower="-3.5" upper="3.5" />
   </joint>
   <!-- chen add -->
